Commit message: Add more calibration targets, adjust camera parameters

File: gz_example/models/landmark/model.sdx.xacro (robot description, xacro)
@@ -5,5 +5,5 @@
         <xacro:property name="size" value="0.03"/>
         <!-- Chessboard size, have to be even numbers -->
-        <xacro:property name="r" value="9"/>
+        <xacro:property name="r" value="8"/>
         <xacro:property name="c" value="7"/>
         <static>true</static>
