Commit message: urdf

File: gz_example/2ur5e/urdf/combined.urdf (robot description, URDF)
Before this commit: robot combined, 53 links, 52 joints
Links:
- removed link ABB1200_base_link
- removed link ABB1200_link_1
- removed link ABB1200_link_2
- removed link ABB1200_link_3
- removed link ABB1200_link_4
- removed link ABB1200_link_5
- removed link ABB1200_link_6
- removed link UR_base_link
- removed link abb_pedestal
- removed link box2-1__body
- removed link box2-2__body
- removed link controller_box
- removed link conveyor__belt
- removed link conveyor__body
- removed link forearm_link
- removed link head
- removed link head_camera
- removed link pedestal
- removed link pedestal_feet
- removed link right_arm_base_link
- removed link right_arm_itb
- removed link right_hand
- removed link right_hand_camera
- removed link right_l0
- removed link right_l1
- removed link right_l1_2
- removed link right_l2
- removed link right_l2_2
- removed link right_l3
- removed link right_l4
- removed link right_l4_2
- removed link right_l5
- removed link right_l6
- removed link right_torso_itb
- removed link right_wrist
- removed link sawyer_pedestal
- removed link screen
- removed link shoulder_link
- removed link torso
- removed link tx60_base_link
- removed link tx60_link_1
- removed link tx60_link_2
- removed link tx60_link_3
- removed link tx60_link_4
- removed link tx60_link_5
- removed link tx60_link_6
- removed link tx60_pedestal
- removed link upper_arm_link
- removed link ur_pedestal
- removed link wrist_1_link
- removed link wrist_2_link
- removed link wrist_3_link
- added link ur5e1__base_link, mass 4; collision mesh filename=model://ur5e/meshes/collision/base.stl scale=1 1 1; visual mesh filename=model://ur5e/meshes/visual/base.dae scale=1 1 1
- added link ur5e1__forearm_link, mass 2.275; collision mesh filename=model://ur5e/meshes/collision/forearm.stl scale=1 1 1; visual mesh filename=model://ur5e/meshes/visual/forearm.stl scale=1 1 1
- added link ur5e1__link_0, mass 1; visual cylinder length=1 radius=0.15
- added link ur5e1__shoulder_link, mass 3.7; collision mesh filename=model://ur5e/meshes/collision/shoulder.stl scale=1 1 1; visual mesh filename=model://ur5e/meshes/visual/shoulder.dae scale=1 1 1
- added link ur5e1__upper_arm_link, mass 8.393; collision mesh filename=model://ur5e/meshes/collision/upperarm.stl scale=1 1 1; visual mesh filename=model://ur5e/meshes/visual/upperarm.stl scale=1 1 1
- added link ur5e1__wrist_1_link, mass 1.219; collision mesh filename=model://ur5e/meshes/collision/wrist1.stl scale=1 1 1; visual mesh filename=model://ur5e/meshes/visual/wrist1.stl scale=1 1 1
- added link ur5e1__wrist_2_link, mass 1.219; collision mesh filename=model://ur5e/meshes/collision/wrist2.stl scale=1 1 1; visual mesh filename=model://ur5e/meshes/visual/wrist2.dae scale=1 1 1
- added link ur5e1__wrist_3_link, mass 0.1879; collision mesh filename=model://ur5e/meshes/collision/wrist3.stl scale=1 1 1; visual mesh filename=model://ur5e/meshes/visual/wrist3.dae scale=1 1 1
- added link ur5e2__base_link, mass 4; collision mesh filename=model://ur5e/meshes/collision/base.stl scale=1 1 1; visual mesh filename=model://ur5e/meshes/visual/base.dae scale=1 1 1
- added link ur5e2__forearm_link, mass 2.275; collision mesh filename=model://ur5e/meshes/collision/forearm.stl scale=1 1 1; visual mesh filename=model://ur5e/meshes/visual/forearm.stl scale=1 1 1
- added link ur5e2__link_0, mass 1; visual cylinder length=1 radius=0.15
- added link ur5e2__shoulder_link, mass 3.7; collision mesh filename=model://ur5e/meshes/collision/shoulder.stl scale=1 1 1; visual mesh filename=model://ur5e/meshes/visual/shoulder.dae scale=1 1 1
- added link ur5e2__upper_arm_link, mass 8.393; collision mesh filename=model://ur5e/meshes/collision/upperarm.stl scale=1 1 1; visual mesh filename=model://ur5e/meshes/visual/upperarm.stl scale=1 1 1
- added link ur5e2__wrist_1_link, mass 1.219; collision mesh filename=model://ur5e/meshes/collision/wrist1.stl scale=1 1 1; visual mesh filename=model://ur5e/meshes/visual/wrist1.stl scale=1 1 1
- added link ur5e2__wrist_2_link, mass 1.219; collision mesh filename=model://ur5e/meshes/collision/wrist2.stl scale=1 1 1; visual mesh filename=model://ur5e/meshes/visual/wrist2.dae scale=1 1 1
- added link ur5e2__wrist_3_link, mass 0.1879; collision mesh filename=model://ur5e/meshes/collision/wrist3.stl scale=1 1 1; visual mesh filename=model://ur5e/meshes/visual/wrist3.dae scale=1 1 1
Joints:
- removed joint ABB1200_joint_1
- removed joint ABB1200_joint_2
- removed joint ABB1200_joint_3
- removed joint ABB1200_joint_4
- removed joint ABB1200_joint_5
- removed joint ABB1200_joint_6
- removed joint abb_pedestal_JOINT_0
- removed joint abb_pose
- removed joint box2-1_joint
- removed joint box2-2_joint
- removed joint controller_box_fixed
- removed joint conveyor__belt_joint
- removed joint conveyor_joint
- removed joint display_joint
- removed joint elbow_joint
- removed joint head_camera
- removed joint head_pan
- removed joint pedestal_feet_fixed
- removed joint pedestal_fixed
- removed joint right_arm_itb
- removed joint right_arm_mount
- removed joint right_hand
- removed joint right_hand_camera
- removed joint right_j0
- removed joint right_j1
- removed joint right_j1_2
- removed joint right_j2
- removed joint right_j2_2
- removed joint right_j3
- removed joint right_j4
- removed joint right_j4_2
- removed joint right_j5
- removed joint right_j6
- removed joint right_torso_itb
- removed joint right_wrist
- removed joint sawyer_pose
- removed joint shoulder_lift_joint
- removed joint shoulder_pan_joint
- removed joint staubli_pose
- removed joint torso_t0
- removed joint tx60_joint_1
- removed joint tx60_joint_2
- removed joint tx60_joint_3
- removed joint tx60_joint_4
- removed joint tx60_joint_5
- removed joint tx60_joint_6
- removed joint tx60_pedestal_JOINT_0
- removed joint ur_pedestal_JOINT_1
- removed joint ur_pose
- removed joint wrist_1_joint
- removed joint wrist_2_joint
- removed joint wrist_3_joint
- added joint ur5e1__elbow_joint: type revolute, parent ur5e1__upper_arm_link, child ur5e1__forearm_link, origin xyz=-0.425  0     0 rpy=0 0 0, axis 0 0 1, limit lower=-3.14159 upper=3.14159 effort=150.0 velocity=3.14159
- added joint ur5e1__link_0_JOINT_1: type fixed, parent ur5e1__link_0, child ur5e1__base_link, origin xyz=0 0 0 rpy=0      0      3.14159, axis 0 0 0, limit lower=0 upper=0 effort=0 velocity=0
- added joint ur5e1__shoulder_lift_joint: type revolute, parent ur5e1__shoulder_link, child ur5e1__upper_arm_link, origin xyz=0 0 0 rpy=1.5708 0     0, axis 0 0 1, limit lower=-6.28319 upper=6.28319 effort=150.0 velocity=3.14159
- added joint ur5e1__shoulder_pan_joint: type revolute, parent ur5e1__base_link, child ur5e1__shoulder_link, origin xyz=0     0     0.1625 rpy=0       0      -3.14159, axis 0 0 1, limit lower=-6.28319 upper=6.28319 effort=150.0 velocity=3.14159
- added joint ur5e1__wrist_1_joint: type revolute, parent ur5e1__forearm_link, child ur5e1__wrist_1_link, origin xyz=-0.3922   0       0.13329 rpy=0 0 0, axis 0 0 1, limit lower=-6.28319 upper=6.28319 effort=28.0 velocity=3.14159
- added joint ur5e1__wrist_2_joint: type revolute, parent ur5e1__wrist_1_link, child ur5e1__wrist_2_link, origin xyz=0     -0.0997  0 rpy=1.57079 0      0, axis 0 0 1, limit lower=-6.28319 upper=6.28319 effort=28.0 velocity=3.14159
- added joint ur5e1__wrist_3_joint: type revolute, parent ur5e1__wrist_2_link, child ur5e1__wrist_3_link, origin xyz=0     0.0996 0 rpy=-1.57079  0       0, axis 0 0 1, limit lower=-6.28319 upper=6.28319 effort=28.0 velocity=3.14159
- added joint ur5e1_pose: type fixed, parent world, child ur5e1__link_0, origin xyz=0 1.2 0.0 rpy=0.0 0.0 0.0
- added joint ur5e2__elbow_joint: type revolute, parent ur5e2__upper_arm_link, child ur5e2__forearm_link, origin xyz=-0.425  0     0 rpy=0 0 0, axis 0 0 1, limit lower=-3.14159 upper=3.14159 effort=150.0 velocity=3.14159
- added joint ur5e2__link_0_JOINT_1: type fixed, parent ur5e2__link_0, child ur5e2__base_link, origin xyz=0 0 0 rpy=0      0      3.14159, axis 0 0 0, limit lower=0 upper=0 effort=0 velocity=0
- added joint ur5e2__shoulder_lift_joint: type revolute, parent ur5e2__shoulder_link, child ur5e2__upper_arm_link, origin xyz=0 0 0 rpy=1.5708 0     0, axis 0 0 1, limit lower=-6.28319 upper=6.28319 effort=150.0 velocity=3.14159
- added joint ur5e2__shoulder_pan_joint: type revolute, parent ur5e2__base_link, child ur5e2__shoulder_link, origin xyz=0     0     0.1625 rpy=0       0      -3.14159, axis 0 0 1, limit lower=-6.28319 upper=6.28319 effort=150.0 velocity=3.14159
- added joint ur5e2__wrist_1_joint: type revolute, parent ur5e2__forearm_link, child ur5e2__wrist_1_link, origin xyz=-0.3922   0       0.13329 rpy=0 0 0, axis 0 0 1, limit lower=-6.28319 upper=6.28319 effort=28.0 velocity=3.14159
- added joint ur5e2__wrist_2_joint: type revolute, parent ur5e2__wrist_1_link, child ur5e2__wrist_2_link, origin xyz=0     -0.0997  0 rpy=1.57079 0      0, axis 0 0 1, limit lower=-6.28319 upper=6.28319 effort=28.0 velocity=3.14159
- added joint ur5e2__wrist_3_joint: type revolute, parent ur5e2__wrist_2_link, child ur5e2__wrist_3_link, origin xyz=0     0.0996 0 rpy=-1.57079  0       0, axis 0 0 1, limit lower=-6.28319 upper=6.28319 effort=28.0 velocity=3.14159
- added joint ur5e2_pose: type fixed, parent world, child ur5e2__link_0, origin xyz=0 0.0 0.0 rpy=0.0 0.0 0.0

Commit message: table

File: gz_example/2ur5e/urdf/combined.urdf (robot description, URDF)
Before this commit: robot combined, 17 links, 16 joints
Links:
- added link table__link, mass 0; collision box size=1.5 0.8 0.03; collision cylinder length=1 radius=0.02
Joints:
- added joint table_pose: type fixed, parent world, child table__link, origin xyz=0 0.0 0.0 rpy=0 0 1.57
